File: Kicad/Sidebar.kicad_pcb (KiCad board)
At the start: 2 copper layers, 84 x 37.7 mm, 8 parts, among them J1 Conn_02x03_Odd_Even, J2 Screw_Power, U1 PY32F002AA15M

Commit message: Updated Kicad Files
Parts:
- added J3: Conn_01x02_Pin, Connector_PinHeader_2.54mm:PinHeader_1x02_P2.54mm_Vertical, B.Cu at (122.5, 119.8)
- R2: value R_US -> 1M
- U1: footprint Package_SO:SSOP-10_3.9x4.9mm_P1.00mm -> Grange:SSOP-10_3.9x4.9mm_P1.00mm
- moved J1 2.55 mm to (134.5, 120.8)
- moved C1 2.41 mm to (129.2, 116.5), turned to 180 degrees
- moved R2 0.75 mm to (143.0, 113.2), turned to 90 degrees
- moved D1 0.20 mm to (142.5, 104.2)
Connections:
- D2 pad 2: Net-(D2-A) -> Net-(D1-A)
- R2 pad 1: Net-(U1-PA6) -> Net-(U1-PA7)
- R2 pad 2: Net-(D2-A) -> SENSE
- U1 pad 2: unconnected-(U1-SDA-Pad2) -> SDA
- U1 pad 3: unconnected-(U1-SCL-Pad3) -> SCL
- U1 pad 6: Net-(U1-PA6) -> SENSE
- U1 pad 7: unconnected-(U1-PA7-Pad7) -> Net-(U1-PA7)
Routing:
- net SCL: track 0.00 -> 14.0 mm
- net SDA: track 0.00 -> 11.5 mm
- net Net-(D2-A): track 9.32 -> 0.00 mm
- net Net-(D1-A): track 5.81 -> 14.4 mm
- net SENSE: track 0.00 -> 5.68 mm, vias 0 -> 1
- net Net-(U1-PA7): track 0.00 -> 5.06 mm
- net Net-(U1-PA6): track 4.52 -> 0.00 mm
- net +3.3V: track 33.0 -> 35.7 mm
- net RST: track 7.93 -> 7.39 mm
- net Net-(J1-Pin_6): track 6.16 -> 5.63 mm
- net Net-(J1-Pin_4): track 7.60 -> 7.06 mm
Other:
- board text added: "SCL"
- board text added: "SDA"
