File: Kicad/Sidebar.kicad_sch (KiCad schematic)
At the start: 8 parts, among them J1 Conn_02x03_Odd_Even, J2 Screw_Power, U1 PY32F002AA15M

Commit message: Updated Kicad Files
Parts:
- added J3: Conn_01x02_Pin, Connector_PinHeader_2.54mm:PinHeader_1x02_P2.54mm_Vertical, symbol Connector:Conn_01x02_Pin
- R2: value R_US -> 1M
- U1: footprint Package_SO:SSOP-10_3.9x4.9mm_P1.00mm -> Grange:SSOP-10_3.9x4.9mm_P1.00mm
Connections:
- net SDA: now reaches U1.2 (SDA)
- net SDA: now also J3.2 (Pin_2)
- net SCL: now reaches U1.3 (SCL)
- net SCL: now also J3.1 (Pin_1)
- net at R2.1: now also U1.7 (PA7); no longer U1.6 (PA6)
- net at D2.2 (A): now also D1.2 (A), R1.1; no longer R2.2
- new net SENSE: R2.2, U1.6 (PA6)
Other:
- title: SaintCon RE Topper -> (none)
- moved on the sheet: D2
